File: ELEC3885_ui.kicad_sch (KiCad schematic)
At the start: 80 parts, among them SW10 RotaryEncoder_Switch, SW11 RotaryEncoder_Switch, SW12 RotaryEncoder_Switch, SW13 RotaryEncoder_Switch, SW14 SW_Push, SW15 SW_Push, SW16 SW_Push, SW17 SW_Push, SW2 SW_Push, SW3 SW_Push, SW4 SW_Push, SW5 SW_Push, SW6 SW_Push, SW7 SW_Push, SW8 SW_Push, SW9 SW_Push, U10 74HC595, U11 LCD_Conn, U8 74HC595, U9 74HC595

Commit message: Rev4 started, changing packages
Parts:
- U10, U8, U9: footprint Package_SO:SOP-16_4.4x10.4mm_P1.27mm -> Package_SO:SOP-16_3.9x9.9mm_P1.27mm
Changed lines of the file:
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@@
       (effects (font (size 1.27 1.27)) (justify left))
     )
-    (property "Footprint" "Package_SO:SOP-16_4.4x10.4mm_P1.27mm" (at 94.615 39.37 0)
+    (property "Footprint" "Package_SO:SOP-16_3.9x9.9mm_P1.27mm" (at 94.615 39.37 0)
       (effects (font (size 1.27 1.27)) hide)
     )
@@
       (effects (font (size 1.27 1.27)) (justify left))
     )
-    (property "Footprint" "Package_SO:SOP-16_4.4x10.4mm_P1.27mm" (at 94.615 82.55 0)
+    (property "Footprint" "Package_SO:SOP-16_3.9x9.9mm_P1.27mm" (at 94.615 82.55 0)
       (effects (font (size 1.27 1.27)) hide)
     )
@@
       (effects (font (size 1.27 1.27)) (justify left))
     )
-    (property "Footprint" "Package_SO:SOP-16_4.4x10.4mm_P1.27mm" (at 94.615 127 0)
-      (effects (font (size 1.27 1.27)) hide)
-    )
+    (property "Footprint" "Package_SO:SOP-16_3.9x9.9mm_P1.27mm" (at 94.615 127 0)
+      (effects (font (size 1.27 1.27)) hide)
+    )
